File: rib.kicad_sch (KiCad schematic)
At the start: 96 parts, among them J1 RJ45_LED, J10 Conn_01x04_Male, J11 Screw_Terminal_01x02, J12 Screw_Terminal_01x02, J13 Screw_Terminal_01x02, J14 Conn_01x02_Male, J15 Conn_01x02_Male, J16 Conn_01x06_Male, J17 Conn_01x02_Male, J18 Conn_01x02_Male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

Commit message: Updated to new version of KiCAD
Parts:
- U2: symbol LM2592HVT:LM2592HVT-3.3/NOPB -> LM2592HVT:LM2592HVT-3.3/NOPB
